File: DI2C/C-RIO_breakout.brd (EAGLE design)
At the start: 105.4 x 103.2 mm, 18 parts, among them X2 0446200002, X4 0446200002

Commit message: update schmeatic
Parts:
- removed X2, X4: 0446200002, con-molex:0446200002
- added R10, R7, R8, R9: 600Ohm, resistor:0414/15
- added T1, T2, T3, T4: 2N2222, transistor-neu-to92:TO18
- added TOF1, TOF2, TOF3, TOF4, U$6: RJ45-8N4-B, con-amphenol-rj45-ld:RJ45-8N4-B
- added X1: (no value), con-subd:F37HP
Connections:
- net N$2 renamed SCL1
- net N$6 renamed SDA1
- net N$7 renamed SCL2
- net N$8 renamed SDA2
- removed net N$1: R1.1, R2.2, U$1.DSCLP, X2.3
- removed net N$3: R2.1, R3.2, U$1.DSCLM, X2.4
- removed net N$5: R5.1, R6.2, U$1.DSDAM, X2.8
- new net DSCLM1: R2.1, R3.2, TOF1.7, TOF2.7, TOF3.7, TOF4.7, U$1.DSCLM
- new net DSCLP1: R1.1, R2.2, TOF1.3, TOF2.3, TOF3.3, TOF4.3, U$1.DSCLP
- new net DSDAM1: R5.1, R6.2, TOF1.2, TOF2.2, TOF3.2, TOF4.2, U$1.DSDAM
- new net DSDAP1: TOF1.5, TOF2.5, TOF3.5, TOF4.5
- new net GND2: TOF1.GND1, TOF1.GND2, TOF2.GND1, TOF2.GND2, TOF3.GND1, TOF3.GND2, TOF4.GND1, TOF4.GND2
- net GND: now also T1.1, T1.3, T2.1, T2.3, T3.1, T3.3, T4.1, T4.3, TOF1.4, TOF1.6, TOF1.8, TOF2.4, TOF2.6, TOF2.8, TOF3.4, TOF3.6, TOF3.8, TOF4.4, TOF4.6, TOF4.8, U$6.2, U$6.5, U$6.8, U$6.GND1, U$6.GND2; no longer X2.2, X2.5, X2.7, X4.2, X4.5, X4.7
- net N$11: now also U$6.3; no longer X4.3
- net N$12: now also U$6.4; no longer X4.4
- net N$15: now also U$6.6; no longer X4.6
- net N$16: now also U$6.7; no longer X4.8
- net N$4: no longer X2.6
- net VDD: now also R10.1, R10.2, R7.1, R7.2, R8.1, R8.2, R9.1, R9.2, TOF1.1, TOF2.1, TOF3.1, TOF4.1, U$6.1; no longer X2.1, X4.1
Routing:
- net GND: track 234.0 -> 0.00 mm
- net N$9: track 209.1 -> 0.00 mm
- net VDD: track 161.3 -> 0.00 mm
- net N$5: track 84.1 -> 0.00 mm
- net N$16: track 80.5 -> 0.00 mm
- net N$15: track 78.7 -> 0.00 mm
- net N$4: track 77.9 -> 0.00 mm
- net N$1: track 77.4 -> 0.00 mm
- net N$11: track 75.0 -> 0.00 mm
- net N$3: track 73.7 -> 0.00 mm
- net N$12: track 72.6 -> 0.00 mm
- net SCL2: track 13.3 -> 0.00 mm
- net SCL1: track 13.0 -> 0.00 mm
- net SDA2: track 10.1 -> 0.00 mm
- net SDA1: track 9.84 -> 0.00 mm
Other:
- board text removed: "High Frequency Channel I2C"
- board text removed: "Low Frequency Channel I2C"

Commit message: added the lsave board
Parts:
- added COMMON: RJ45-8N4-B, con-amphenol-rj45-ld:RJ45-8N4-B
- added SV1: (no value), con-lstb:MA06-1
- added X2, X3: (no value), con-wago-508:W237-8P
- moved T1 320.5 mm to (48.4, 155.4), flipped to the bottom
- moved T2 320.5 mm to (48.4, 139.4), flipped to the bottom
- moved T3 320.5 mm to (48.4, 123.4), flipped to the bottom
- moved T4 320.5 mm to (48.4, 107.4), flipped to the bottom
- moved TOF4 293.8 mm to (90.0, 161.0), turned to 90 degrees
- moved R10 282.1 mm to (63.0, 137.0), turned to 90 degrees
- moved R9 265.7 mm to (62.0, 113.0), turned to 90 degrees
- moved X1 261.2 mm to (3.08, 21.2), flipped to the bottom, turned to 270 degrees
- moved TOF3 241.8 mm to (90.0, 139.0), turned to 90 degrees
- moved R8 212.2 mm to (70.0, 137.0), turned to 270 degrees
- moved TOF1 179.2 mm to (90.0, 118.0), turned to 90 degrees
- moved R7 147.1 mm to (69.0, 113.0), turned to 270 degrees
Connections:
- new net AI0: X1.7, X2.1
- new net AI1: X1.8, X2.2
- new net AI2: X1.9, X2.3
- new net AI3: X1.10, X2.4
- new net AI4: X1.11, X2.5
- new net AI5: X1.12, X2.6
- new net AI6: X1.13, X2.7
- new net AI7: X1.14, X2.8
- new net AO0: X1.1, X3.1
- new net AO1: X1.2, X3.2
- new net AO2: X1.21, X3.3
- new net AO3: X1.22, X3.4
- new net AO4: X1.4, X3.5
- new net AO5: X1.5, X3.6
- new net AO6: X1.24, X3.7
- new net AO7: X1.25, X3.8
- new net DIO0: T3.2, X1.15
- new net DIO1: T4.2, X1.16
- new net DIO2: T2.2, X1.17
- new net DIO3: T1.2, X1.18
- new net GNDT1: T1.3, TOF4.8
- new net GNDT2: T2.3, TOF3.8
- new net GNDT3: T3.3, TOF1.8
- new net GNDT4: T4.3, TOF2.8
- net DSCLM1: now also COMMON.7
- net DSCLP1: now also COMMON.3
- net DSDAM1: now also COMMON.2
- net DSDAP1: now also COMMON.5
- net GND: now also COMMON.4, COMMON.6, COMMON.8, COMMON.GND1, COMMON.GND2, SV1.2, X1.19, X1.20, X1.23, X1.26, X1.27, X1.28, X1.29, X1.3, X1.30, X1.31, X1.32, X1.33, X1.34, X1.35, X1.36, X1.37, X1.6; no longer T1.3, T2.3, T3.3, T4.3, TOF1.8, TOF2.8, TOF3.8, TOF4.8
- net SCL1: now also SV1.3
- net SDA1: now also SV1.4
- net VDD: now also COMMON.1, SV1.1
Routing:
- net GND: track 0.00 -> 550.0 mm
- net VDD: track 0.00 -> 444.0 mm, vias 0 -> 1
- net DIO3: track 0.00 -> 177.7 mm
- net DSCLM1: track 0.00 -> 164.5 mm
- net DSDAM1: track 0.00 -> 164.4 mm
- net DSCLP1: track 0.00 -> 162.8 mm, vias 0 -> 1
- net DIO2: track 0.00 -> 157.9 mm
- net DIO0: track 0.00 -> 136.8 mm
- net DIO1: track 0.00 -> 122.8 mm
- net SCL1: track 0.00 -> 113.8 mm
- net SDA1: track 0.00 -> 106.0 mm
- net AI7: track 0.00 -> 93.5 mm
- net AI6: track 0.00 -> 92.5 mm
- net AI5: track 0.00 -> 91.6 mm
- net AI4: track 0.00 -> 90.6 mm
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Other:
- board size 105.4 x 103.2 mm -> 110.5 x 222.7 mm
- board text added: "Analog In"
- board text added: "Analog Out"
- board text added: "Current Sensor"
- board text added: "TOF"
- board text added: "Universal"
